File: WeatherStationSender/WeatherStationSender.sch (KiCad schematic (older format))
At the start: 4 parts

Commit message: finished pcb for order
Parts:
- added J2: Conn_01x02_Male, Connector_PinSocket_2.54mm:PinSocket_1x02_P2.54mm_Vertical, symbol Connector:Conn_01x02_Male
- J1: renamed from J?; footprint (none) -> Connector_PinHeader_2.54mm:PinHeader_1x03_P2.54mm_Vertical
- U1: renamed from U?; footprint (none) -> Package_TO_SOT_THT:TO-220F-3_Horizontal_TabDown
- gave numbers to parts that had none: 2
Connections:
- net GND: now also A1.29 (GND), A1.4 (GND), J2.2 (Pin_2)
- net +9V: now reaches A1.30 (VIN)
- net +9V: now also J2.1 (Pin_1)
Changed lines of the file:
@@
 $EndDescr
 $Comp
-L MCU_Module:Arduino_Nano_v3.x A?
+L MCU_Module:Arduino_Nano_v3.x A1
 U 1 1 5E3F5EAB
 P 5600 3700
-F 0 "A?" H 5600 2611 50  0000 C CNN
+F 0 "A1" H 5600 2611 50  0000 C CNN
 F 1 "Arduino_Nano_v3.x" H 5600 2520 50  0000 C CNN
 F 2 "Module:Arduino_Nano" H 5600 3700 50  0001 C CIN
@@
 $EndComp
 $Comp
-L Regulator_Linear:AZ1117-3.3 U?
+L Regulator_Linear:AZ1117-3.3 U1
 U 1 1 5E3F68B8
 P 7350 4350
-F 0 "U?" H 7350 4592 50  0000 C CNN
+F 0 "U1" H 7350 4592 50  0000 C CNN
 F 1 "AZ1117-3.3" H 7350 4501 50  0000 C CNN
-F 2 "" H 7350 4600 50  0001 C CIN
+F 2 "Package_TO_SOT_THT:TO-220F-3_Horizontal_TabDown" H 7350 4600 50  0001 C CIN
 F 3 "https://www.diodes.com/assets/Datasheets/AZ1117.pdf" H 7350 4350 50  0001 C CNN
 	1    7350 4350
@@
 $EndComp
 $Comp
-L RF:NRF24L01_Breakout U?
+L RF:NRF24L01_Breakout U2
 U 1 1 5E3F6FDC
 P 7450 3050
-F 0 "U?" H 7830 3096 50  0000 L CNN
+F 0 "U2" H 7830 3096 50  0000 L CNN
 F 1 "NRF24L01_Breakout" H 7830 3005 50  0000 L CNN
 F 2 "RF_Module:nRF24L01_Breakout" H 7600 3650 50  0001 L CIN
@@
 $EndComp
 $Comp
-L power:+5V #PWR?
+L power:+5V #PWR0101
 U 1 1 5E3F95DE
 P 3200 3350
-F 0 "#PWR?" H 3200 3200 50  0001 C CNN
+F 0 "#PWR0101" H 3200 3200 50  0001 C CNN
 F 1 "+5V" H 3215 3523 50  0000 C CNN
 F 2 "" H 3200 3350 50  0001 C CNN
@@
 $EndComp
 $Comp
-L Connector:Conn_01x03_Female J?
+L Connector:Conn_01x03_Female J1
 U 1 1 5E3F8423
 P 3300 3150
-F 0 "J?" V 3238 2962 50  0000 R CNN
+F 0 "J1" V 3238 2962 50  0000 R CNN
 F 1 "Conn_01x03_Female" V 3147 2962 50  0000 R CNN
-F 2 "" H 3300 3150 50  0001 C CNN
+F 2 "Connector_PinHeader_2.54mm:PinHeader_1x03_P2.54mm_Vertical" H 3300 3150 50  0001 C CNN
 F 3 "~" H 3300 3150 50  0001 C CNN
 	1    3300 3150
@@
 DHT_DATA
 $Comp
-L power:GND #PWR?
+L power:GND #PWR0102
 U 1 1 5E3F9F2A
 P 3400 3350
-F 0 "#PWR?" H 3400 3100 50  0001 C CNN
+F 0 "#PWR0102" H 3400 3100 50  0001 C CNN
 F 1 "GND" H 3405 3177 50  0000 C CNN
 F 2 "" H 3400 3350 50  0001 C CNN
@@
 $EndComp
 $Comp
-L power:+5V #PWR?
+L power:+5V #PWR0103
 U 1 1 5E3FBBA3
 P 5800 2700
-F 0 "#PWR?" H 5800 2550 50  0001 C CNN
+F 0 "#PWR0103" H 5800 2550 50  0001 C CNN
 F 1 "+5V" H 5815 2873 50  0000 C CNN
 F 2 "" H 5800 2700 50  0001 C CNN
@@
 NRF_ENABLE
 $Comp
-L power:+3.3V #PWR?
+L power:+3.3V #PWR0104
 U 1 1 5E3FC56E
 P 7450 2450
-F 0 "#PWR?" H 7450 2300 50  0001 C CNN
+F 0 "#PWR0104" H 7450 2300 50  0001 C CNN
 F 1 "+3.3V" H 7465 2623 50  0000 C CNN
 F 2 "" H 7450 2450 50  0001 C CNN
@@
 $EndComp
 $Comp
-L power:GND #PWR?
+L power:GND #PWR0105
 U 1 1 5E3FCECA
 P 7450 3650
-F 0 "#PWR?" H 7450 3400 50  0001 C CNN
+F 0 "#PWR0105" H 7450 3400 50  0001 C CNN
 F 1 "GND" H 7455 3477 50  0000 C CNN
 F 2 "" H 7450 3650 50  0001 C CNN
@@
 $EndComp
 $Comp
-L power:GND #PWR?
+L power:GND #PWR0106
 U 1 1 5E3FD05F
 P 7350 4650
-F 0 "#PWR?" H 7350 4400 50  0001 C CNN
+F 0 "#PWR0106" H 7350 4400 50  0001 C CNN
 F 1 "GND" H 7355 4477 50  0000 C CNN
 F 2 "" H 7350 4650 50  0001 C CNN
@@
 $EndComp
 $Comp
-L power:+3.3V #PWR?
+L power:+3.3V #PWR0107
 U 1 1 5E3FD273
 P 7650 4350
-F 0 "#PWR?" H 7650 4200 50  0001 C CNN
+F 0 "#PWR0107" H 7650 4200 50  0001 C CNN
 F 1 "+3.3V" V 7665 4478 50  0000 L CNN
 F 2 "" H 7650 4350 50  0001 C CNN
@@
 $EndComp
 $Comp
-L power:+5V #PWR?
+L power:+5V #PWR0108
 U 1 1 5E3FD46B
 P 7050 4350
-F 0 "#PWR?" H 7050 4200 50  0001 C CNN
+F 0 "#PWR0108" H 7050 4200 50  0001 C CNN
 F 1 "+5V" V 7065 4478 50  0000 L CNN
 F 2 "" H 7050 4350 50  0001 C CNN
@@
 Text HLabel 5100 4000 0    50   Input ~ 0
 NRF_ENABLE
+$Comp
+L Connector:Conn_01x02_Male J2
+U 1 1 5E407AB9
+P 4450 2450
+F 0 "J2" V 4512 2494 50  0000 L CNN
+F 1 "Conn_01x02_Male" V 4603 2494 50  0000 L CNN
+F 2 "Connector_PinSocket_2.54mm:PinSocket_1x02_P2.54mm_Vertical" H 4450 2450 50  0001 C CNN
+F 3 "~" H 4450 2450 50  0001 C CNN
+	1    4450 2450
+	0    1    1    0
+$EndComp
+$Comp
+L power:GND #PWR0109
+U 1 1 5E408771
+P 4350 2650
+F 0 "#PWR0109" H 4350 2400 50  0001 C CNN
+F 1 "GND" H 4355 2477 50  0000 C CNN
+F 2 "" H 4350 2650 50  0001 C CNN
+F 3 "" H 4350 2650 50  0001 C CNN
+	1    4350 2650
+	1    0    0    -1
+$EndComp
+$Comp
+L power:+9V #PWR0110
+U 1 1 5E408AFA
+P 4450 2650
+F 0 "#PWR0110" H 4450 2500 50  0001 C CNN
+F 1 "+9V" H 4465 2823 50  0000 C CNN
+F 2 "" H 4450 2650 50  0001 C CNN
+F 3 "" H 4450 2650 50  0001 C CNN
+	1    4450 2650
+	-1   0    0    1
+$EndComp
+$Comp
+L power:+9V #PWR0111
+U 1 1 5E409009
+P 5500 2700
+F 0 "#PWR0111" H 5500 2550 50  0001 C CNN
+F 1 "+9V" H 5515 2873 50  0000 C CNN
+F 2 "" H 5500 2700 50  0001 C CNN
+F 3 "" H 5500 2700 50  0001 C CNN
+	1    5500 2700
+	1    0    0    -1
+$EndComp
+$Comp
+L power:GND #PWR?
+U 1 1 5E40D34C
+P 5600 4700
+F 0 "#PWR?" H 5600 4450 50  0001 C CNN
+F 1 "GND" H 5605 4527 50  0000 C CNN
+F 2 "" H 5600 4700 50  0001 C CNN
+F 3 "" H 5600 4700 50  0001 C CNN
+	1    5600 4700
+	1    0    0    -1
+$EndComp
+$Comp
+L power:GND #PWR?
+U 1 1 5E40D587
+P 5700 4700
+F 0 "#PWR?" H 5700 4450 50  0001 C CNN
+F 1 "GND" H 5705 4527 50  0000 C CNN
+F 2 "" H 5700 4700 50  0001 C CNN
+F 3 "" H 5700 4700 50  0001 C CNN
+	1    5700 4700
+	1    0    0    -1
+$EndComp
 $EndSCHEMATC
